Commit message: Fixed wrong indent size for xacro/xml files.

File: sfg_go2_description/xacro/constants.xacro (robot description, xacro)
@@ -1,26 +1,26 @@
 <?xml version="1.0"?>
 <robot xmlns:xacro="http://www.ros.org/wiki/xacro">
-    <!-- offset of the thigh along the x and y axes relative to the base -->
-    <xacro:property name="hip_offset_x" value="0.1934" />
-    <xacro:property name="hip_offset_y" value="0.0465" />
-    <!-- offset of the thigh along y axis relative to the hip -->
-    <xacro:property name="thigh_offset_y" value="0.0955" />
-    <!-- lengths of leg components -->
-    <xacro:property name="thigh_length" value="0.213" />
-    <xacro:property name="calf_length" value="0.213" />
-    <!-- hip joint limits -->
-    <xacro:property name="hip_position_max" value="1.0472" />
-    <xacro:property name="hip_position_min" value="-1.0472" />
-    <xacro:property name="hip_velocity_max" value="30.1" />
-    <xacro:property name="hip_torque_max" value="23.7" />
-    <!-- thigh joint limits -->
-    <xacro:property name="thigh_position_max" value="3.4907" />
-    <xacro:property name="thigh_position_min" value="-1.5708" />
-    <xacro:property name="thigh_velocity_max" value="30.1" />
-    <xacro:property name="thigh_torque_max" value="23.7" />
-    <!-- calf joint limits -->
-    <xacro:property name="calf_position_max" value="-0.83776" />
-    <xacro:property name="calf_position_min" value="-2.7227" />
-    <xacro:property name="calf_velocity_max" value="20.06" />
-    <xacro:property name="calf_torque_max" value="35.55" />
+  <!-- offset of the thigh along the x and y axes relative to the base -->
+  <xacro:property name="hip_offset_x" value="0.1934" />
+  <xacro:property name="hip_offset_y" value="0.0465" />
+  <!-- offset of the thigh along y axis relative to the hip -->
+  <xacro:property name="thigh_offset_y" value="0.0955" />
+  <!-- lengths of leg components -->
+  <xacro:property name="thigh_length" value="0.213" />
+  <xacro:property name="calf_length" value="0.213" />
+  <!-- hip joint limits -->
+  <xacro:property name="hip_position_max" value="1.0472" />
+  <xacro:property name="hip_position_min" value="-1.0472" />
+  <xacro:property name="hip_velocity_max" value="30.1" />
+  <xacro:property name="hip_torque_max" value="23.7" />
+  <!-- thigh joint limits -->
+  <xacro:property name="thigh_position_max" value="3.4907" />
+  <xacro:property name="thigh_position_min" value="-1.5708" />
+  <xacro:property name="thigh_velocity_max" value="30.1" />
+  <xacro:property name="thigh_torque_max" value="23.7" />
+  <!-- calf joint limits -->
+  <xacro:property name="calf_position_max" value="-0.83776" />
+  <xacro:property name="calf_position_min" value="-2.7227" />
+  <xacro:property name="calf_velocity_max" value="20.06" />
+  <xacro:property name="calf_torque_max" value="35.55" />
 </robot>

File: sfg_go2_description/xacro/leg.xacro (robot description, xacro)
@@ -1,66 +1,66 @@
 <?xml version="1.0"?>
 <robot xmlns:xacro="http://www.ros.org/wiki/xacro">
-    <xacro:macro name="leg" params="name front left">
-        <joint name="${name}_hip_joint" type="revolute">
-            <parent link="base" />
-            <child link="${name}_hip" />
-            <origin rpy="0 0 0" xyz="${front * hip_offset_x} ${left * hip_offset_y} 0" />
-            <axis xyz="1 0 0" />
-            <xacro:if value="${left == 1}">
-                <limit effort="${hip_torque_max}" velocity="${hip_velocity_max}"
-                    lower="${hip_position_min}" upper="${hip_position_max}" />
-            </xacro:if>
-            <xacro:if value="${left == -1}">
-                <limit effort="${hip_torque_max}" velocity="${hip_velocity_max}"
-                    lower="${-hip_position_max}" upper="${-hip_position_min}" />
-            </xacro:if>
-        </joint>
-        <link name="${name}_hip">
-            <visual>
-                <origin rpy="${(1 - left) / 2 * pi} ${(1 - front) / 2 * pi} 0" xyz="0 0 0 " />
-                <geometry>
-                    <mesh filename="package://sfg_go2_description/mesh/hip.dae"
-                        scale="1 1 1" />
-                </geometry>
-            </visual>
-        </link>
-        <joint name="${name}_thigh_joint" type="revolute">
-            <parent link="${name}_hip" />
-            <child link="${name}_thigh" />
-            <origin rpy="0 0 0" xyz="0 ${left * thigh_offset_y} 0" />
-            <axis xyz="0 1 0" />
-            <limit effort="${thigh_torque_max}" velocity="${thigh_velocity_max}"
-                lower="${thigh_position_min}" upper="${thigh_position_max}" />
-        </joint>
-        <link name="${name}_thigh">
-            <visual>
-                <geometry>
-                    <mesh filename="package://sfg_go2_description/mesh/thigh.dae"
-                        scale="1 ${left} 1" />
-                </geometry>
-            </visual>
-        </link>
-        <joint name="${name}_calf_joint" type="revolute">
-            <parent link="${name}_thigh" />
-            <child link="${name}_calf" />
-            <origin rpy="0 0 0" xyz="0 0 ${-thigh_length}" />
-            <axis xyz="0 1 0" />
-            <limit effort="${calf_torque_max}" velocity="${calf_velocity_max}"
-                lower="${calf_position_min}" upper="${calf_position_max}" />
-        </joint>
-        <link name="${name}_calf">
-            <visual>
-                <geometry>
-                    <mesh filename="package://sfg_go2_description/mesh/calf.dae"
-                        scale="1 ${left} 1" />
-                </geometry>
-            </visual>
-        </link>
-        <joint name="${name}_foot_joint" type="fixed">
-            <parent link="${name}_calf" />
-            <child link="${name}_foot" />
-            <origin rpy="0 0 0" xyz="0 0 ${-calf_length}" />
-        </joint>
-        <link name="${name}_foot" />
-    </xacro:macro>
+  <xacro:macro name="leg" params="name front left">
+    <joint name="${name}_hip_joint" type="revolute">
+      <parent link="base" />
+      <child link="${name}_hip" />
+      <origin rpy="0 0 0" xyz="${front * hip_offset_x} ${left * hip_offset_y} 0" />
+      <axis xyz="1 0 0" />
+      <xacro:if value="${left == 1}">
+        <limit effort="${hip_torque_max}" velocity="${hip_velocity_max}"
+          lower="${hip_position_min}" upper="${hip_position_max}" />
+      </xacro:if>
+      <xacro:if value="${left == -1}">
+        <limit effort="${hip_torque_max}" velocity="${hip_velocity_max}"
+          lower="${-hip_position_max}" upper="${-hip_position_min}" />
+      </xacro:if>
+    </joint>
+    <link name="${name}_hip">
+      <visual>
+        <origin rpy="${(1 - left) / 2 * pi} ${(1 - front) / 2 * pi} 0" xyz="0 0 0 " />
+        <geometry>
+          <mesh filename="package://sfg_go2_description/mesh/hip.dae"
+            scale="1 1 1" />
+        </geometry>
+      </visual>
+    </link>
+    <joint name="${name}_thigh_joint" type="revolute">
+      <parent link="${name}_hip" />
+      <child link="${name}_thigh" />
+      <origin rpy="0 0 0" xyz="0 ${left * thigh_offset_y} 0" />
+      <axis xyz="0 1 0" />
+      <limit effort="${thigh_torque_max}" velocity="${thigh_velocity_max}"
+        lower="${thigh_position_min}" upper="${thigh_position_max}" />
+    </joint>
+    <link name="${name}_thigh">
+      <visual>
+        <geometry>
+          <mesh filename="package://sfg_go2_description/mesh/thigh.dae"
+            scale="1 ${left} 1" />
+        </geometry>
+      </visual>
+    </link>
+    <joint name="${name}_calf_joint" type="revolute">
+      <parent link="${name}_thigh" />
+      <child link="${name}_calf" />
+      <origin rpy="0 0 0" xyz="0 0 ${-thigh_length}" />
+      <axis xyz="0 1 0" />
+      <limit effort="${calf_torque_max}" velocity="${calf_velocity_max}"
+        lower="${calf_position_min}" upper="${calf_position_max}" />
+    </joint>
+    <link name="${name}_calf">
+      <visual>
+        <geometry>
+          <mesh filename="package://sfg_go2_description/mesh/calf.dae"
+            scale="1 ${left} 1" />
+        </geometry>
+      </visual>
+    </link>
+    <joint name="${name}_foot_joint" type="fixed">
+      <parent link="${name}_calf" />
+      <child link="${name}_foot" />
+      <origin rpy="0 0 0" xyz="0 0 ${-calf_length}" />
+    </joint>
+    <link name="${name}_foot" />
+  </xacro:macro>
 </robot>

File: sfg_go2_description/xacro/robot_description.urdf.xacro (robot description, xacro)
@@ -1,61 +1,61 @@
 <?xml version="1.0"?>
 <robot name="go2" xmlns:xacro="http://www.ros.org/wiki/xacro">
-    <xacro:include filename="$(find sfg_go2_description)/xacro/constants.xacro" />
-    <xacro:include filename="$(find sfg_go2_description)/xacro/leg.xacro" />
-    <xacro:include filename="$(find sfg_peripherals_description)/xacro/htc_vive_tracker_30.xacro" />
-    <xacro:include filename="$(find sfg_peripherals_description)/xacro/intel_realsense_d435.xacro" />
-    <xacro:include filename="$(find sfg_peripherals_description)/xacro/livox_mid360.xacro" />
-    <link name="base">
-        <visual>
-            <geometry>
-                <mesh filename="package://sfg_go2_description/mesh/base.dae" scale="1 1 1" />
-            </geometry>
-        </visual>
-    </link>
-    <!-- legs -->
-    <xacro:leg name="front_left" front="1" left="1" />
-    <xacro:leg name="front_right" front="1" left="-1" />
-    <xacro:leg name="rear_left" front="-1" left="1" />
-    <xacro:leg name="rear_right" front="-1" left="-1" />
-    <!-- head assembly mount -->
-    <joint name="head_assembly_mount_joint" type="fixed">
-        <parent link="base" />
-        <child link="head_assembly_mount" />
-        <origin rpy="0 0.10074 0" xyz="0.24797 0 0.0807" />
-    </joint>
-    <link name="head_assembly_mount">
-        <visual>
-            <geometry>
-                <mesh
-                    filename="package://sfg_go2_description/mesh/head_assembly_mount.dae"
-                    scale="1 1 1" />
-            </geometry>
-        </visual>
-    </link>
-    <!-- camera head -->
-    <xacro:intel_realsense_d435 name="camera_head" parent="head_assembly_mount">
-        <origin rpy="0 ${0.5 * pi} 0" xyz="0.06081 0.00001 0.00946" />
-    </xacro:intel_realsense_d435>
-    <!-- tracker head -->
-    <xacro:htc_vive_tracker_30 name="tracker_head" parent="head_assembly_mount">
-        <origin rpy="0 0 0" xyz="0 0 0.0337" />
-    </xacro:htc_vive_tracker_30>
-    <!-- extension dock -->
-    <joint name="extension_dock_joint" type="fixed">
-        <parent link="base" />
-        <child link="extension_dock" />
-        <origin rpy="0 0 0" xyz="-0.01896 0 0.05699" />
-    </joint>
-    <link name="extension_dock">
-        <visual>
-            <geometry>
-                <mesh filename="package://sfg_go2_description/mesh/extension_dock.dae"
-                    scale="1 1 1" />
-            </geometry>
-        </visual>
-    </link>
-    <!-- lidar back -->
-    <xacro:livox_mid360 name="lidar_back" parent="extension_dock">
-        <origin rpy="0 0 ${pi}" xyz="-0.0531 0 0.0537" />
-    </xacro:livox_mid360>
+  <xacro:include filename="$(find sfg_go2_description)/xacro/constants.xacro" />
+  <xacro:include filename="$(find sfg_go2_description)/xacro/leg.xacro" />
+  <xacro:include filename="$(find sfg_peripherals_description)/xacro/htc_vive_tracker_30.xacro" />
+  <xacro:include filename="$(find sfg_peripherals_description)/xacro/intel_realsense_d435.xacro" />
+  <xacro:include filename="$(find sfg_peripherals_description)/xacro/livox_mid360.xacro" />
+  <link name="base">
+    <visual>
+      <geometry>
+        <mesh filename="package://sfg_go2_description/mesh/base.dae" scale="1 1 1" />
+      </geometry>
+    </visual>
+  </link>
+  <!-- legs -->
+  <xacro:leg name="front_left" front="1" left="1" />
+  <xacro:leg name="front_right" front="1" left="-1" />
+  <xacro:leg name="rear_left" front="-1" left="1" />
+  <xacro:leg name="rear_right" front="-1" left="-1" />
+  <!-- head assembly mount -->
+  <joint name="head_assembly_mount_joint" type="fixed">
+    <parent link="base" />
+    <child link="head_assembly_mount" />
+    <origin rpy="0 0.10074 0" xyz="0.24797 0 0.0807" />
+  </joint>
+  <link name="head_assembly_mount">
+    <visual>
+      <geometry>
+        <mesh
+          filename="package://sfg_go2_description/mesh/head_assembly_mount.dae"
+          scale="1 1 1" />
+      </geometry>
+    </visual>
+  </link>
+  <!-- camera head -->
+  <xacro:intel_realsense_d435 name="camera_head" parent="head_assembly_mount">
+    <origin rpy="0 ${0.5 * pi} 0" xyz="0.06081 0.00001 0.00946" />
+  </xacro:intel_realsense_d435>
+  <!-- tracker head -->
+  <xacro:htc_vive_tracker_30 name="tracker_head" parent="head_assembly_mount">
+    <origin rpy="0 0 0" xyz="0 0 0.0337" />
+  </xacro:htc_vive_tracker_30>
+  <!-- extension dock -->
+  <joint name="extension_dock_joint" type="fixed">
+    <parent link="base" />
+    <child link="extension_dock" />
+    <origin rpy="0 0 0" xyz="-0.01896 0 0.05699" />
+  </joint>
+  <link name="extension_dock">
+    <visual>
+      <geometry>
+        <mesh filename="package://sfg_go2_description/mesh/extension_dock.dae"
+          scale="1 1 1" />
+      </geometry>
+    </visual>
+  </link>
+  <!-- lidar back -->
+  <xacro:livox_mid360 name="lidar_back" parent="extension_dock">
+    <origin rpy="0 0 ${pi}" xyz="-0.0531 0 0.0537" />
+  </xacro:livox_mid360>
 </robot>
