Commit message: sfg_go2_description: Added anti vibration tracker mount.

File: sfg_go2_description/xacro/robot_description.urdf.xacro (robot description, xacro)
@@ -39,5 +39,5 @@
     <!-- tracker -->
     <xacro:htc_vive_tracker_30 name="tracker" parent="head_assembly_mount">
-        <origin rpy="0 0 0" xyz="0 0 0.016" />
+        <origin rpy="0 0 0" xyz="0 0 0.0337" />
     </xacro:htc_vive_tracker_30>
     <!-- extension dock -->

Commit message: sfg_go2_description: use path relative includes for all includes in robot_description.urdf.xacro.

File: sfg_go2_description/xacro/robot_description.urdf.xacro (robot description, xacro)
@@ -1,6 +1,6 @@
 <?xml version="1.0"?>
 <robot name="go2" xmlns:xacro="http://www.ros.org/wiki/xacro">
-    <xacro:include filename="constants.xacro" />
-    <xacro:include filename="leg.xacro" />
+    <xacro:include filename="$(find sfg_go2_description)/xacro/constants.xacro" />
+    <xacro:include filename="$(find sfg_go2_description)/xacro/leg.xacro" />
     <xacro:include filename="$(find sfg_peripherals_description)/xacro/htc_vive_tracker_30.xacro" />
     <xacro:include filename="$(find sfg_peripherals_description)/xacro/intel_realsense_d435.xacro" />
@@ -57,5 +57,5 @@
     <!-- lidar back -->
     <xacro:livox_mid360 name="lidar_back" parent="extension_dock">
-        <origin rpy="0 0 0" xyz="-0.0531 0 0.0537" />
+        <origin rpy="0 0 ${pi}" xyz="-0.0531 0 0.0537" />
     </xacro:livox_mid360>
 </robot>

Commit message: sfg_go2_description: Updated robot description to include base marker tree instead of htc vive tracker.

File: sfg_go2_description/xacro/robot_description.urdf.xacro (robot description, xacro)
@@ -3,5 +3,5 @@
   <xacro:include filename="$(find sfg_go2_description)/xacro/constants.xacro" />
   <xacro:include filename="$(find sfg_go2_description)/xacro/leg.xacro" />
-  <xacro:include filename="$(find sfg_peripherals_description)/xacro/htc_vive_tracker_30.xacro" />
+  <xacro:include filename="$(find sfg_peripherals_description)/xacro/base_marker_tree.xacro" />
   <xacro:include filename="$(find sfg_peripherals_description)/xacro/intel_realsense_d435.xacro" />
   <xacro:include filename="$(find sfg_peripherals_description)/xacro/livox_mid360.xacro" />
@@ -38,7 +38,7 @@
   </xacro:intel_realsense_d435>
   <!-- tracker head -->
-  <xacro:htc_vive_tracker_30 name="tracker_head" parent="head_assembly_mount">
-    <origin rpy="0 0 0" xyz="0 0 0.0337" />
-  </xacro:htc_vive_tracker_30>
+  <xacro:base_marker_tree name="tracker_head" parent="head_assembly_mount">
+    <origin rpy="0 0 0" xyz="0 0 0.01396" />
+  </xacro:base_marker_tree>
   <!-- extension dock -->
   <joint name="extension_dock_joint" type="fixed">

Commit message: Created robot_description.xacro, an actual macro to make the whole description reusable.

File: sfg_go2_description/xacro/robot_description.urdf.xacro (robot description, xacro)
@@ -1,61 +1,7 @@
 <?xml version="1.0"?>
 <robot name="go2" xmlns:xacro="http://www.ros.org/wiki/xacro">
-  <xacro:include filename="$(find sfg_go2_description)/xacro/constants.xacro" />
-  <xacro:include filename="$(find sfg_go2_description)/xacro/leg.xacro" />
-  <xacro:include filename="$(find sfg_peripherals_description)/xacro/base_marker_tree.xacro" />
-  <xacro:include filename="$(find sfg_peripherals_description)/xacro/intel_realsense_d435.xacro" />
-  <xacro:include filename="$(find sfg_peripherals_description)/xacro/livox_mid360.xacro" />
-  <link name="base">
-    <visual>
-      <geometry>
-        <mesh filename="package://sfg_go2_description/mesh/base.dae" scale="1 1 1" />
-      </geometry>
-    </visual>
-  </link>
-  <!-- legs -->
-  <xacro:leg name="front_left" front="1" left="1" />
-  <xacro:leg name="front_right" front="1" left="-1" />
-  <xacro:leg name="rear_left" front="-1" left="1" />
-  <xacro:leg name="rear_right" front="-1" left="-1" />
-  <!-- head assembly mount -->
-  <joint name="head_assembly_mount_joint" type="fixed">
-    <parent link="base" />
-    <child link="head_assembly_mount" />
-    <origin rpy="0 0.10074 0" xyz="0.24797 0 0.0807" />
-  </joint>
-  <link name="head_assembly_mount">
-    <visual>
-      <geometry>
-        <mesh
-          filename="package://sfg_go2_description/mesh/head_assembly_mount.dae"
-          scale="1 1 1" />
-      </geometry>
-    </visual>
-  </link>
-  <!-- camera head -->
-  <xacro:intel_realsense_d435 name="camera_head" parent="head_assembly_mount">
-    <origin rpy="0 ${0.5 * pi} 0" xyz="0.06081 0.00001 0.00946" />
-  </xacro:intel_realsense_d435>
-  <!-- tracker head -->
-  <xacro:base_marker_tree name="tracker_head" parent="head_assembly_mount">
-    <origin rpy="0 0 0" xyz="0 0 0.01396" />
-  </xacro:base_marker_tree>
-  <!-- extension dock -->
-  <joint name="extension_dock_joint" type="fixed">
-    <parent link="base" />
-    <child link="extension_dock" />
-    <origin rpy="0 0 0" xyz="-0.01896 0 0.05699" />
-  </joint>
-  <link name="extension_dock">
-    <visual>
-      <geometry>
-        <mesh filename="package://sfg_go2_description/mesh/extension_dock.dae"
-          scale="1 1 1" />
-      </geometry>
-    </visual>
-  </link>
-  <!-- lidar back -->
-  <xacro:livox_mid360 name="lidar_back" parent="extension_dock">
-    <origin rpy="0 0 ${pi}" xyz="-0.0531 0 0.0537" />
-  </xacro:livox_mid360>
+  <xacro:include filename="$(find sfg_go2_description)/xacro/robot_description.xacro" />
+  <xacro:go2_robot_description>
+    <origin rpy="0 0 0" xyz="0 0 0" />
+  </xacro:go2_robot_description>
 </robot>
