Commit message: sfg_go2_description: Replace .dae with .glb meshes.

File: sfg_go2_description/xacro/leg.xacro (robot description, xacro)
@@ -3,7 +3,7 @@
   <xacro:macro name="leg" params="name front left">
     <joint name="${name}_hip_joint" type="revolute">
-      <parent link="base" />
+      <parent link="base_link" />
       <child link="${name}_hip" />
-      <origin rpy="0 0 0" xyz="${front * hip_offset_x} ${left * hip_offset_y} 0" />
+      <origin xyz="${front * hip_offset_x} ${left * hip_offset_y} 0" rpy="0 0 0" />
       <axis xyz="1 0 0" />
       <xacro:if value="${left == 1}">
@@ -18,7 +18,7 @@
     <link name="${name}_hip">
       <visual>
-        <origin rpy="${(1 - left) / 2 * pi} ${(1 - front) / 2 * pi} 0" xyz="0 0 0 " />
+        <origin xyz="0 0 0" rpy="${(1 - left) / 2 * pi + left * 0.5 * pi} ${(1 - front) / 2 * pi} 0" />
         <geometry>
-          <mesh filename="package://sfg_go2_description/mesh/hip.dae"
+          <mesh filename="package://sfg_go2_description/mesh/hip.glb"
             scale="1 1 1" />
         </geometry>
@@ -28,5 +28,5 @@
       <parent link="${name}_hip" />
       <child link="${name}_thigh" />
-      <origin rpy="0 0 0" xyz="0 ${left * thigh_offset_y} 0" />
+      <origin xyz="0 ${left * thigh_offset_y} 0" rpy="0 0 0" />
       <axis xyz="0 1 0" />
       <limit effort="${thigh_torque_max}" velocity="${thigh_velocity_max}"
@@ -35,6 +35,7 @@
     <link name="${name}_thigh">
       <visual>
+        <origin xyz="0 0 0" rpy="${left * 0.5 * pi} 0 0" />
         <geometry>
-          <mesh filename="package://sfg_go2_description/mesh/thigh.dae"
+          <mesh filename="package://sfg_go2_description/mesh/thigh.glb"
             scale="1 ${left} 1" />
         </geometry>
@@ -44,5 +45,5 @@
       <parent link="${name}_thigh" />
       <child link="${name}_calf" />
-      <origin rpy="0 0 0" xyz="0 0 ${-thigh_length}" />
+      <origin xyz="0 0 ${-thigh_length}" rpy="0 0 0" />
       <axis xyz="0 1 0" />
       <limit effort="${calf_torque_max}" velocity="${calf_velocity_max}"
@@ -51,6 +52,7 @@
     <link name="${name}_calf">
       <visual>
+        <origin xyz="0 0 0" rpy="${left * 0.5 * pi} 0 0" />
         <geometry>
-          <mesh filename="package://sfg_go2_description/mesh/calf.dae"
+          <mesh filename="package://sfg_go2_description/mesh/calf.glb"
             scale="1 ${left} 1" />
         </geometry>
@@ -60,5 +62,5 @@
       <parent link="${name}_calf" />
       <child link="${name}_foot" />
-      <origin rpy="0 0 0" xyz="0 0 ${-calf_length}" />
+      <origin xyz="0 0 ${-calf_length}" rpy="0 0 0" />
     </joint>
     <link name="${name}_foot" />

File: sfg_go2_description/xacro/robot_description.xacro (robot description, xacro)
@@ -1,5 +1,5 @@
 <?xml version="1.0"?>
 <robot name="go2" xmlns:xacro="http://www.ros.org/wiki/xacro">
-  <xacro:macro name="go2_robot_description" params="name:='base' parent:='' *origin">
+  <xacro:macro name="go2_robot_description" params="name:='base_link' parent:='' *origin">
     <xacro:include filename="$(find sfg_go2_description)/xacro/constants.xacro" />
     <xacro:include filename="$(find sfg_go2_description)/xacro/leg.xacro" />
@@ -16,6 +16,7 @@
     <link name="${name}">
       <visual>
+        <origin xyz="0 0 0" rpy="${0.5 * pi} 0 0" />
         <geometry>
-          <mesh filename="package://sfg_go2_description/mesh/base.dae" scale="1 1 1" />
+          <mesh filename="package://sfg_go2_description/mesh/base_link.glb" />
         </geometry>
       </visual>
@@ -30,12 +31,12 @@
       <parent link="${name}" />
       <child link="head_assembly_mount" />
-      <origin rpy="0 0.10074 0" xyz="0.24797 0 0.0807" />
+      <origin xyz="0.24797 0 0.0807" rpy="0 0.10074 0" />
     </joint>
     <link name="head_assembly_mount">
       <visual>
+        <origin xyz="0 0 0" rpy="${0.5 * pi} 0 ${0.5 * pi}" />
         <geometry>
           <mesh
-            filename="package://sfg_go2_description/mesh/head_assembly_mount.dae"
-            scale="1 1 1" />
+            filename="package://sfg_go2_description/mesh/head_assembly_mount.glb" />
         </geometry>
       </visual>
@@ -43,9 +44,9 @@
     <!-- camera head -->
     <xacro:intel_realsense_d435 name="camera_head" parent="head_assembly_mount">
-      <origin rpy="0 ${0.5 * pi} 0" xyz="0.06081 0.00001 0.00946" />
+      <origin xyz="0.06081 0.00001 0.00946" rpy="0 ${0.5 * pi} 0" />
     </xacro:intel_realsense_d435>
     <!-- tracker head -->
     <xacro:base_marker_tree name="tracker_head" parent="head_assembly_mount">
-      <origin rpy="0 0 0" xyz="0 0 0.01396" />
+      <origin xyz="0 0 0.01396" rpy="0 0 0" />
     </xacro:base_marker_tree>
     <!-- extension dock -->
@@ -53,11 +54,11 @@
       <parent link="${name}" />
       <child link="extension_dock" />
-      <origin rpy="0 0 0" xyz="-0.01896 0 0.05699" />
+      <origin xyz="-0.01896 0 0.05699" rpy="0 0 0" />
     </joint>
     <link name="extension_dock">
       <visual>
+        <origin xyz="0 0 0" rpy="${0.5 * pi} 0 ${0.5 * pi}" />
         <geometry>
-          <mesh filename="package://sfg_go2_description/mesh/extension_dock.dae"
-            scale="1 1 1" />
+          <mesh filename="package://sfg_go2_description/mesh/extension_dock.glb" />
         </geometry>
       </visual>
@@ -65,5 +66,5 @@
     <!-- lidar back -->
     <xacro:livox_mid360 name="lidar_back" parent="extension_dock">
-      <origin rpy="0 0 ${pi}" xyz="-0.0531 0 0.0537" />
+      <origin xyz="-0.0531 0 0.0537" rpy="0 0 ${pi}" />
     </xacro:livox_mid360>
   </xacro:macro>

Commit message: sfg_go2_description: Removed default scale in xacro files.

File: sfg_go2_description/xacro/leg.xacro (robot description, xacro)
@@ -20,6 +20,5 @@
         <origin xyz="0 0 0" rpy="${(1 - left) / 2 * pi + left * 0.5 * pi} ${(1 - front) / 2 * pi} 0" />
         <geometry>
-          <mesh filename="package://sfg_go2_description/mesh/hip.glb"
-            scale="1 1 1" />
+          <mesh filename="package://sfg_go2_description/mesh/hip.glb" />
         </geometry>
       </visual>

Commit message: sfg_go2_description: Fix for wrong hip orientation on right side.

File: sfg_go2_description/xacro/leg.xacro (robot description, xacro)
@@ -18,5 +18,5 @@
     <link name="${name}_hip">
       <visual>
-        <origin xyz="0 0 0" rpy="${(1 - left) / 2 * pi + left * 0.5 * pi} ${(1 - front) / 2 * pi} 0" />
+        <origin xyz="0 0 0" rpy="${-(1 - left) * pi + left * 0.5 * pi} ${(1 - front) / 2 * pi} 0" />
         <geometry>
           <mesh filename="package://sfg_go2_description/mesh/hip.glb" />
